Commit message: better car popping

File: control_tree_car/urdf/car.urdf (robot description, URDF)
Before this commit: robot lgp_car, 1 links, 0 joints
Links:
- link lgp_car: geometry visual mesh filename=package://control_tree_car/meshes/bmw/G12Pos8.dae

Commit message: update car model

File: control_tree_car/urdf/car.urdf (robot description, URDF)
Before this commit: robot lgp_car, 1 links, 0 joints
Links:
- link lgp_car: geometry visual mesh filename=package://control_tree_car/meshes/bmw/bmw.dae
